File: Hardware/Electronics/Eagle/Liploft_Schematics.sch (EAGLE design)
At the start: 13 parts, among them U1 MCP4161, U2 MCP4161, U3 MCP4161, U4 MCP4161

Commit message: Updated the schematics
Connections:
- new net N$14: BL.CTS-I, BL.RTS-O
Changed lines of the file:
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@@
+</segment>
+</net>
+<net name="N$14" class="0">
+<segment>
+<pinref part="BL" gate="G$1" pin="CTS-I"/>
+<wire x1="-53.34" y1="127" x2="-50.8" y2="127" width="0.1524" layer="91"/>
+<wire x1="-50.8" y1="127" x2="-50.8" y2="116.84" width="0.1524" layer="91"/>
+<pinref part="BL" gate="G$1" pin="RTS-O"/>
+<wire x1="-50.8" y1="116.84" x2="-53.34" y2="116.84" width="0.1524" layer="91"/>
 </segment>
 </net>
